File: hw/boards/tp1/tp1.kicad_sch (KiCad schematic)
At the start: 24 parts

Commit message: TK-1 and TP-1 PCBs (#52)
* Add kicad library for flat programming clip

* Add descriptions to part symbols

* Add extended values, manufacturer/distributor info to components in mta1

* Add new board entry for TK1

* Add TP1 programmer design

* Update MTA1-USB-V1 release files to match production

* Change SPI flash memory type to XT25F08BDFIGT-S
* Change touch sensor feedback cap to 1uF
* Add manufacturer, manufacturer part number, distributor, distributor part number

* Update component values for TK1 PCB

* Use specific part # for C8
* Change flash back to Winbond part, for easier sourcing
* Change C1 to 1pF

* Fixes for production programmer PCB

* Swap GND and 5V on J3
* Replace graphic logo with text
* Rename part to 'TP-1'

* TK-1 release

* Add dimensions for PCB
* Add layer stackup for PCB
* Change PCB component origin to match expanded board
* Change schematic title to 'TK-1', update release date

* mta1-usb-v1-programmer: Add corrected part numbers for OSFC production

* Q1, Q2, F1 part subsititutions
* add mfr/supplier info for all parts

* PCB library: add parts

* Rectangular footprint for TK-1 test pads
* BOM generation script used for TK-1 and TP-1 releases

* TP-1 release

* Schematic: Add manufacturer, supplier information for all parts
* Schematic: Update name and release date
* PCB: Add PCB fabrication information
* PCB: Correct pinouts on silkscreen

* PCB library: add 'screw' and 'foot' symbols

* Screw is a schematic-only part, for including mechanical screws in the
  BOM
* Foot is for self-adhesive rubber mounting feet that can be stuck to
  the bottom of a PCB

* TP-1 release: Add screws, feet to the BOM

* Pico library: Add footprint for RPi Pico w/solder paste

* TP-1 RevA release updates:

* Add fiducials in 3 corners (1mm exposed copper ring w/2mm soldermask opening)
* Add solder paste openings to Raspberry Pi Pico pads

* TK-1: RevA.1 release

* Add two fiducials to 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
Parts:
- removed R1, R10, R2, R3, R4, R5, R6, R9: (no value), symbol Device:R
- removed U1: (no value), symbol mta1:mta1_usb_ch554_pogo
- added FID1, FID2, FID3: (no value), symbol Mechanical:Fiducial
- added FOOT1, FOOT2, FOOT3, FOOT4: (no value), symbol mta1:Foot
- added J3: (no value), symbol mta1:BC-1-208
- added J4: (no value), symbol mta1:BC-1-701
- added SCREW1, SCREW2, SCREW3: (no value), symbol mta1:Screw
- F1: Manufacturer RUILON -> Littelfuse; Manufacturer Part Number SMD1206P005TF -> 1206L005/60WR; Supplier lcsc -> Digikey; Supplier Part Number C20797 -> F8129TR-ND
- J1, J2: now left out of the parts list
- Q1: Manufacturer winsok -> Alpha & Omega; Manufacturer Part Number WST3400A -> AO3400A; Supplier lcsc -> Digikey; Supplier Part Number C2758406 -> 785-1000-2-ND
- Q2: Extended Value 1%,1/16W -> (none); Manufacturer jjm -> Alpha & Omega; Manufacturer Part Number JMTL3401A -> AO3401A; Supplier lcsc -> Digikey; Supplier Part Number C394037 -> 785-1001-2-ND
- R11, R12, R13, R14, R15, R16, R17: Extended Value (none) -> 1/16W,5%; Manufacturer yageo -> Any/not critical; Manufacturer Part Number AF0402FR-07100RL -> (none); Supplier Digikey -> (none); Supplier Part Number 13-AF0402FR-07100RLTR-ND -> (none)
- R7, R8: Extended Value 1%,1/16W -> 1/16W,5%; Manufacturer yageo -> Any/not critical; Manufacturer Part Number AT0402FRE0710KL -> (none); Supplier Digikey -> (none); Supplier Part Number YAG2104TR-ND -> (none)
Connections:
- net 5V_DUT: now also J3.1
- net CDONE: now also J4.6
- net CRESET: now also J4.5
- net GND: now also J3.2, J4.7
- net MISO: now also J4.4
- net MOSI: now also J4.2
- net SCK: now also J4.1
- net SS: now also J4.3
- net +1V2 renamed PICO26
- net +2V5 renamed PICO27
- net +3V3 renamed PICO28
Other:
- note added: "Note: J1 and J2 are DNP"
- note added: "Tillitis TK-1 Programmer (TP-1)"
- note removed: "MTA1-USB-V1 Programmer"
- title: mta1-usb-v1-programmer -> Tillits TK1 Programmer (TP-1)
