File: prototypes/mta1-usb-v1-programmer/mta1-usb-v1-programmer.kicad_sch (KiCad schematic)
At the start: 24 parts

Commit message: Update links to library and 3D-models for the prototype mta1-usb-v1-programmer.
Parts:
- F1: value (none) -> 50mA, nSMD005; footprint (none) -> Fuse:Fuse_1206_3216Metric
- J1, J2: value (none) -> Conn_01x20; footprint (none) -> Connector_PinHeader_2.54mm:PinHeader_1x20_P2.54mm_Vertical
- Q1: value (none) -> WST3400A; footprint (none) -> Package_TO_SOT_SMD:SOT-23
- Q2: value (none) -> JMTL3401A; footprint (none) -> Package_TO_SOT_SMD:SOT-23
- R1, R10, R11, R12, R13, R14, R15, R16, R17, R2, R3, R4, R5, R6, R9: value (none) -> R100; footprint (none) -> mta1:ERJ2G(0402)_L
- R7, R8: value (none) -> 10K; footprint (none) -> mta1:ERJ2G(0402)_L
- U1: value (none) -> mta1_usb_ch554_pogo; footprint (none) -> mta1:mta1_usb_ch554_pogo
- U2: value (none) -> Pico; footprint (none) -> RPi_Pico:RPi_Pico_SMD_TH
Connections:
- net +3V3 renamed +3.3V
